File: attenuverter_v1/attenuverter_block.kicad_sch (KiCad schematic)
At the start: 17 parts, among them U1 TL072

Commit message: Silkscreen cleanup and labeling
Other:
- title: Annetuverter -> Triple Annetuverter
Changed lines of the file:
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@@
   (paper "A4")
   (title_block
-    (title "Annetuverter")
+    (title "Triple Annetuverter")
     (date "2022-07-05")
     (rev "1.0")

Commit message: Geographic rename
Parts:
- renumbered C6 to C100, C5 to C101, C3 to C2, C4 to C3, R3 to R100, R5 to R2, R1 to R3, R8 to R4, R4 to R5, R2 to R8
Changed lines of the file:
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@@
   (symbol (lib_id "Device:C") (at 215.265 97.79 0)
     (in_bom yes) (on_board yes) (fields_autoplaced)
-    (property "Reference" "C5" (id 0) (at 218.186 96.8815 0)
+    (property "Reference" "C101" (id 0) (at 218.186 96.8815 0)
       (effects (font (size 1.27 1.27)) (justify left))
     )
@@
   (symbol (lib_id "Device:C") (at 119.38 116.205 90)
     (in_bom yes) (on_board yes) (fields_autoplaced)
-    (property "Reference" "C4" (id 0) (at 119.38 110.0795 90))
+    (property "Reference" "C3" (id 0) (at 119.38 110.0795 90))
     (property "Value" "10pF" (id 1) (at 119.38 112.8546 90))
     (property "Footprint" "Capacitor_SMD:C_1206_3216Metric_Pad1.33x1.80mm_HandSolder" (id 2) (at 123.19 115.2398 0)
@@
   (symbol (lib_id "Device:R") (at 179.705 94.615 270)
     (in_bom yes) (on_board yes) (fields_autoplaced)
-    (property "Reference" "R2" (id 0) (at 179.705 89.6325 90))
+    (property "Reference" "R8" (id 0) (at 179.705 89.6325 90))
     (property "Value" "1k" (id 1) (at 179.705 92.4076 90))
     (property "Footprint" "Resistor_SMD:R_1206_3216Metric_Pad1.30x1.75mm_HandSolder" (id 2) (at 179.705 92.837 90)
@@
   (symbol (lib_id "Device:R") (at 87.63 94.615 270)
     (in_bom yes) (on_board yes) (fields_autoplaced)
-    (property "Reference" "R1" (id 0) (at 87.63 89.6325 90))
+    (property "Reference" "R3" (id 0) (at 87.63 89.6325 90))
     (property "Value" "100k" (id 1) (at 87.63 92.4076 90))
     (property "Footprint" "Resistor_SMD:R_1206_3216Metric_Pad1.30x1.75mm_HandSolder" (id 2) (at 87.63 92.837 90)
@@
   (symbol (lib_id "Device:R") (at 158.75 104.775 270)
     (in_bom yes) (on_board yes) (fields_autoplaced)
-    (property "Reference" "R5" (id 0) (at 158.75 99.7925 90))
+    (property "Reference" "R2" (id 0) (at 158.75 99.7925 90))
     (property "Value" "10k" (id 1) (at 158.75 102.5676 90))
     (property "Footprint" "Resistor_SMD:R_1206_3216Metric_Pad1.30x1.75mm_HandSolder" (id 2) (at 158.75 102.997 90)
@@
   (symbol (lib_id "Device:C") (at 215.265 106.045 0)
     (in_bom yes) (on_board yes) (fields_autoplaced)
-    (property "Reference" "C6" (id 0) (at 218.186 105.1365 0)
+    (property "Reference" "C100" (id 0) (at 218.186 105.1365 0)
       (effects (font (size 1.27 1.27)) (justify left))
     )
@@
   (symbol (lib_id "Device:C") (at 158.75 113.665 90)
     (in_bom yes) (on_board yes) (fields_autoplaced)
-    (property "Reference" "C3" (id 0) (at 158.75 107.5395 90))
+    (property "Reference" "C2" (id 0) (at 158.75 107.5395 90))
     (property "Value" "10pF" (id 1) (at 158.75 110.3146 90))
     (property "Footprint" "Capacitor_SMD:C_1206_3216Metric_Pad1.33x1.80mm_HandSolder" (id 2) (at 162.56 112.6998 0)
@@
   (symbol (lib_id "Device:R") (at 90.805 112.395 90)
     (in_bom yes) (on_board yes) (fields_autoplaced)
-    (property "Reference" "R8" (id 0) (at 90.805 107.4125 90))
+    (property "Reference" "R4" (id 0) (at 90.805 107.4125 90))
     (property "Value" "100k" (id 1) (at 90.805 110.1876 90))
     (property "Footprint" "Resistor_SMD:R_1206_3216Metric_Pad1.30x1.75mm_HandSolder" (id 2) (at 90.805 114.173 90)
@@
   (symbol (lib_id "Device:R") (at 136.525 97.155 90)
     (in_bom yes) (on_board yes) (fields_autoplaced)
-    (property "Reference" "R3" (id 0) (at 136.525 92.1725 90))
+    (property "Reference" "R100" (id 0) (at 136.525 92.1725 90))
     (property "Value" "10k" (id 1) (at 136.525 94.9476 90))
     (property "Footprint" "Resistor_SMD:R_1206_3216Metric_Pad1.30x1.75mm_HandSolder" (id 2) (at 136.525 98.933 90)
@@
   (symbol (lib_id "Device:R") (at 143.51 100.965 180)
     (in_bom yes) (on_board yes) (fields_autoplaced)
-    (property "Reference" "R4" (id 0) (at 145.288 100.0565 0)
-      (effects (font (size 1.27 1.27)) (justify right))
-    )
+    (property "Reference" "R5" (id 0) (at 145.288 100.0565 0)
+      (effects (font (size 1.27 1.27)) (justify right))
+    )
