File: attenuverter_v1/attenuverter_v1.kicad_pcb (KiCad board)
At the start: 2 copper layers, 38 x 100 mm, 61 parts, among them J1 Conn_02x05_Odd_Even, J2 AudioJack2_SwitchT, J3 AudioJack2_SwitchT, J4 AudioJack2_SwitchT, J5 AudioJack2_SwitchT, J6 AudioJack2_SwitchT, J7 AudioJack2_SwitchT, U1 TL072, U2 TL072, U3 TL072

Commit message: First pass routing done
Parts:
- moved D3 3.16 mm to (162.4, 91.7), turned to 90 degrees
- moved FB2 2.27 mm to (158.6, 91.2), turned to 90 degrees
- moved C14 1.75 mm to (157.7, 141.8)
- moved R23 1.75 mm to (157.7, 144.5)
- moved C4 1.48 mm to (156.8, 69.2)
- moved R7 1.48 mm to (156.8, 66.4)
- moved FB1 0.70 mm to (157.3, 72.5)
- moved D2 0.30 mm to (161.2, 75.0)
Routing:
- net -12V: track 0.00 -> 199.1 mm, vias 0 -> 2
- net +12V: track 0.00 -> 117.2 mm
- net Net-(C3-Pad2): track 0.00 -> 28.7 mm
- net Net-(C9-Pad2): track 0.00 -> 26.8 mm
- net Net-(C13-Pad2): track 0.00 -> 26.7 mm
- net Net-(C14-Pad1): track 0.00 -> 24.3 mm
- net Net-(C10-Pad1): track 0.00 -> 22.2 mm
- net Net-(C4-Pad1): track 0.00 -> 20.6 mm
- net /Attenuverter Block/IN: track 0.00 -> 19.6 mm
- net Net-(ATEN1-Pad3): track 0.00 -> 19.6 mm
- net /Attenuverter Block1/IN: track 0.00 -> 18.7 mm
- net /Attenuverter Block2/IN: track 0.00 -> 18.3 mm
- net +12VA: track 0.00 -> 17.7 mm
- net Net-(C13-Pad1): track 0.00 -> 17.1 mm
- net Net-(C9-Pad1): track 0.00 -> 17.0 mm
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
Commit message: Silkscreen cleanup and labeling
Parts:
- moved LOGO1 123.5 mm to (158.9, 145.5)
- moved LOGO2 114.0 mm to (158.8, 124.9)
- moved LOGO3 77.0 mm to (158.7, 67.9)
Other:
- board text added: "40.64mm = 8HP"
- board text added: "Robot Dialogs"
- board text added: "Triple Attenuverter"
- board text added: "v1.0 July 2022"
- board text removed: "15.24 = 3HP"

Commit message: Geographic rename
Parts:
- renumbered C6 to C100, C5 to C101, C8 to C102, C7 to C103, C12 to C104, C11 to C105, C3 to C2, C4 to C3, C1 to C4, C2 to C5, C9 to C6, C10 to C7, C13 to C8, C14 to C9, D2 to D1, D3 to D2, J1 to J8, LOGO3 to LOGO100, LOGO2 to LOGO101, LOGO1 to LOGO102, R13 to R10, R3 to R100, R11 to R101, R19 to R102, R16 to R11, R14 to R13, R10 to R14, R21 to R16, R24 to R18, R20 to R19, R5 to R2, R22 to R20, R18 to R21, R23 to R22, R1 to R3, R8 to R4, R4 to R5, R2 to R8
